Commit message: camera and lidar added

File: src/my_robot/urdf/my_robot.xacro (robot description, xacro)
@@ -56,5 +56,5 @@
   </link>
 	<link name='left_wheel'>
-		<collission>
+		<collision>
 			<origin xyz="0 0 0" rpy="0 1.5707 1.5707"/>
 			<geometry>
@@ -65,5 +65,5 @@
 			<origin xyz="0 0 0" rpy="0 1.5707 1.5707"/>
 			<mass value = "5"/>
-			<inertia ixx="0.1" ixy="0" ixz="0" iyy="0.1" izz="0" izz="0.1"/>
+			<inertia ixx="0.1" ixy="0" ixz="0" iyy="0.1" iyz="0" izz="0.1"/>
 		</inertial>
 		<visual>
@@ -83,5 +83,5 @@
   </joint>
 	<link name='right_wheel'>
-		<collission>
+		<collision>
 			<origin xyz="0 0 0" rpy="0 1.5707 1.5707"/>
 			<geometry>
@@ -92,5 +92,5 @@
 			<origin xyz="0 0 0" rpy="0 1.5707 1.5707"/>
 			<mass value = "5"/>
-			<inertia ixx="0.1" ixy="0" ixz="0" iyy="0.1" izz="0" izz="0.1"/>
+			<inertia ixx="0.1" ixy="0" ixz="0" iyy="0.1" iyz="0" izz="0.1"/>
 		</inertial>
 		<visual>
@@ -109,3 +109,60 @@
     <dynamics damping="1.0" friction="1.0"/>
   </joint>
+	<link name='camera'>
+		<visual>
+			<origin xyz='0 0 0' rpy='0 0 0'>
+			</origin>
+			<geometry>
+				<box size='0.05 0.05 0.05'/>
+			</geometry>
+		</visual>
+		<inertial>
+			<origin xyz='0 0 0' rpy='0 0 0'>
+			</origin>
+			<mass value='0.05'/>
+			<box_inertia m="0.1" x="0.05" y="0.05" z="0.05"/>
+			<inertia ixx="1e-6" ixy="0" ixz="0" iyy="1e-6" iyz="0" izz="1e-6"/>
+		</inertial>
+		<collision>
+			<origin xyz='0 0 0' rpy='0 0 0'>
+			</origin>
+			<geometry>
+				<box size='0.05 0.05 0.05'/>
+			</geometry>
+		</collision>
+	</link>
+  <joint type="fixed" name="camera_joint">
+    <origin xyz="0.2 0 0" rpy="0 0 0"/>
+    <child link="camera"/>
+    <parent link="chassis"/>
+    <axis xyz="0 1 0"/>
+  </joint>
+	<link name='hokuyo'>
+		<visual>
+			<origin xyz='0 0 0' rpy='0 0 0'>
+			</origin>
+			<geometry>
+				<mesh filename='package://my_robot/meshes/hokuyo.dae'/>
+			</geometry>
+		</visual>
+		<inertial>
+			<origin xyz='0 0 0' rpy='0 0 0'>
+			</origin>
+			<mass value='1e-5'/>
+			<inertia ixx="1e-6" ixy="0" ixz="0" iyy="1e-6" iyz="0" izz="1e-6"/>
+		</inertial>
+		<collision>
+			<origin xyz='0 0 0' rpy='0 0 0'>
+			</origin>
+			<geometry>
+				<box size='0.1 0.1 0.1'/>
+			</geometry>
+		</collision>
+	</link>
+  <joint type="fixed" name="hokuyo_joint">
+    <origin xyz="0.15 0 0.1" rpy="0 0 0"/>
+    <child link="hokuyo"/>
+    <parent link="chassis"/>
+    <axis xyz="0 1 0"/>
+  </joint>
 </robot>

Commit message: Project 1 world added

File: src/my_robot/urdf/my_robot.xacro (robot description, xacro)
@@ -1,4 +1,5 @@
 <?xml version='1.0'?>
 <robot name="my_robot" xmlns:xacro="http://www.ros.org/wiki/xacro">
+  <xacro:include filename="$(find my_robot)/urdf/my_robot.gazebo" />
   <link name="robot_footprint"></link>
   <joint name="robot_footprint_joint" type="fixed">
@@ -166,3 +167,12 @@
     <axis xyz="0 1 0"/>
   </joint>
+	<gazebo reference="left_wheel">
+    <material>Gazebo/Green</material>
+	</gazebo>
+	<gazebo reference="right_wheel">
+    <material>Gazebo/Green</material>
+	</gazebo>
+	<gazebo reference="chasis">
+    <material>Gazebo/Blue</material>
+	</gazebo>
 </robot>
